File: PCI/Circuito3Led.brd (EAGLE design)
At the start: 100 x 80 mm, 7 parts

Commit message: Segundo commit
Parts:
- LED1, LED2, LED3: device led:LUMILED -> led:LED5MM
- R1, R2, R3: device rcl:0207/10 -> rcl:0204/7
- moved R1 18.1 mm to (62.2, 25.4)
- moved LED1 16.6 mm to (58.4, 20.3)
- moved R2 14.2 mm to (52.1, 25.4)
- moved R3 12.7 mm to (41.9, 25.4)
- moved LED2 12.6 mm to (45.7, 20.3)
- moved LED3 9.25 mm to (33.0, 20.3)
- moved U$1 6.48 mm to (48.3, 57.1)
Connections:
- net GND: now also LED1.K, LED2.K, LED3.K, U$1.GND@2; no longer R1.2, R2.2, R3.2
- net N$1: now also R3.1; no longer LED3.2+
- net N$2: now also R2.1; no longer LED2.2+
- net N$3: now also R1.1; no longer LED1.2+
- net N$4: now also LED1.A, R1.2; no longer LED1.4-, R1.1
- net N$5: now also LED2.A, R2.2; no longer LED2.4-, R2.1
- net N$6: now also LED3.A, R3.2; no longer LED3.4-, R3.1
Routing:
- net N$4: track 38.0 -> 11.7 mm
- net N$5: track 36.8 -> 14.3 mm
- net N$6: track 38.1 -> 16.8 mm
- net N$2: track 20.4 -> 26.9 mm
- net GND: track 59.8 -> 65.5 mm
- net N$3: track 30.3 -> 26.3 mm
- net N$1: track 24.4 -> 20.8 mm
