File: PCI/Circuito3Led.sch (EAGLE design)
At the start: 7 parts

Commit message: Segundo commit
Parts:
- LED1, LED2, LED3: device led:LED-LUMILED -> led:LED5MM
- R1, R2, R3: device rcl:R-US_0207/10 -> rcl:R-US_0204/7
Connections:
- net GND: now also LED1.C, LED2.C, LED3.C, U$1.GND@2; no longer R1.2, R2.2, R3.2
- net N$1: now also R3.1; no longer LED3.A
- net N$2: now also R2.1; no longer LED2.A
- net N$3: now also R1.1; no longer LED1.A
- net N$4: now also LED1.A, R1.2; no longer LED1.C, R1.1
- net N$5: now also LED2.A, R2.2; no longer LED2.C, R2.1
- net N$6: now also LED3.A, R3.2; no longer LED3.C, R3.1
Other:
- note added: "R1, R2 e R3 = 330R LED1 = VERMELHOR LED2 = AZUL LED3 = AMARELO"
- moved on the sheet: LED1, LED2, LED3, R1, R2, R3, U$1
